File: HW/carecasetester/carecasetester.kicad_pcb (KiCad board)
At the start: 4 copper layers, 158.3 x 150.4 mm, 37 parts, among them J1 Conn_01x16_Female, J10-TP22 Conn_01x01_Male, J11-TP7 Conn_01x01_Male, J12-TP14 Conn_01x01_Male, J13-TP23 Conn_01x01_Male, J14-TP17 Conn_01x01_Male, J15 Conn_01x16_Male, J15-TP1 Conn_01x01_Male, J15-TP20 Conn_01x01_Male, J16-TP2 Conn_01x01_Male, J16-TP24 Conn_01x01_Male, J17-TP3 Conn_01x01_Male, J18-TP4 Conn_01x01_Male, J19-TP6 Conn_01x01_Male, J2 Conn_01x16_Female, J20-TP9 Conn_01x01_Male, J21-TP10 Conn_01x01_Male, J22-TP11 Conn_01x01_Male, J23-TP12 Conn_01x01_Male, J24-TP15 Conn_01x01_Male, J25-TP18 Conn_01x01_Male, J27-TP26 Conn_01x01_Male, J28-TP5 Conn_01x01_Male, J3 Conn_01x04_Female, J4 Conn_01x06_Male, J4-TP16 Conn_01x01_Male, J5-TP8 Conn_01x01_Male, J5-~E1 Conn_01x02_Male, J6-EXT_PWR1 Conn_01x02_Male, J6-TP21 Conn_01x01_Male, J7-TP27 Conn_01x01_Male, J8-TP13 Conn_01x01_Male, J9-TP19 Conn_01x01_Male, SW1 SW_DIP_x02, U1 CD74HC4067M

Commit message: cc-tester v0.1 gerber filser genereret og 1. print bestilles
Parts:
- removed J28-TP5: Conn_01x01_Male, MM:P50-E-120-G(Pogo)_0.7mmHole_1.5mmPad
- removed J6-EXT_PWR1: Conn_01x02_Male, Connector_PinHeader_2.54mm:PinHeader_1x02_P2.54mm_Vertical
- added C1: 100µf, Capacitor_SMD:C_0603_1608Metric_Pad1.05x0.95mm_HandSolder, F.Cu at (173.6, 39.3)
- added C2: 100nf, Capacitor_SMD:C_0603_1608Metric_Pad1.05x0.95mm_HandSolder, F.Cu at (177.6, 39.3)
- added C3: 100µf, Capacitor_SMD:C_0603_1608Metric_Pad1.05x0.95mm_HandSolder, F.Cu at (175.6, 39.3)
- added D1: 1N4001-B, Diode_THT:D_DO-41_SOD81_P10.16mm_Horizontal, F.Cu at (182.0, 44.6)
- added D2: 1N4148W, Diode_THT:D_DO-35_SOD27_P10.16mm_Horizontal, F.Cu at (233.0, 31.2)
- added J26-TP5: Conn_01x01_Male, MM:P50-E-120-G(Pogo)_0.7mmHole_1.5mmPad, F.Cu at (209.0, 128.7)
- added J5: 12V_Psu, athir:Friwo_Texas_2-pin_Plug(1321609), F.Cu at (180.2, 20.2)
- added K1: AZ952, athir:AZ952, F.Cu at (228.6, 19.9)
- added Q1: BC847, Package_TO_SOT_SMD:SOT-23, F.Cu at (218.2, 36.7)
- added R10: 7k6, Resistor_SMD:R_0603_1608Metric_Pad1.05x0.95mm_HandSolder, F.Cu at (140.7, 42.2)
- added R11: 7k6, Resistor_SMD:R_0603_1608Metric_Pad1.05x0.95mm_HandSolder, F.Cu at (137.9, 42.2)
- added R12: 7k6, Resistor_SMD:R_0603_1608Metric_Pad1.05x0.95mm_HandSolder, F.Cu at (135.1, 42.2)
- added R13: 7k6, Resistor_SMD:R_0603_1608Metric_Pad1.05x0.95mm_HandSolder, F.Cu at (132.4, 42.2)
- added R14: 20k, Resistor_SMD:R_0603_1608Metric_Pad1.05x0.95mm_HandSolder, F.Cu at (162.8, 49.1)
- added R15: 20k, Resistor_SMD:R_0603_1608Metric_Pad1.05x0.95mm_HandSolder, F.Cu at (160.1, 47.0)
- added R16: 3k9, Resistor_SMD:R_0603_1608Metric_Pad1.05x0.95mm_HandSolder, F.Cu at (157.2, 49.2)
- added R17: 2k9, Resistor_SMD:R_0603_1608Metric_Pad1.05x0.95mm_HandSolder, F.Cu at (154.5, 49.2)
- added R18: 2k9, Resistor_SMD:R_0603_1608Metric_Pad1.05x0.95mm_HandSolder, F.Cu at (151.7, 49.2)
- added R19: 3k9, Resistor_SMD:R_0603_1608Metric_Pad1.05x0.95mm_HandSolder, F.Cu at (148.9, 49.2)
- added R2: 7k6, Resistor_SMD:R_0603_1608Metric_Pad1.05x0.95mm_HandSolder, F.Cu at (162.9, 42.2)
- added R20: 3k9, Resistor_SMD:R_0603_1608Metric_Pad1.05x0.95mm_HandSolder, F.Cu at (146.1, 49.3)
- added R21: 20k, Resistor_SMD:R_0603_1608Metric_Pad1.05x0.95mm_HandSolder, F.Cu at (143.3, 49.2)
- added R22: 20k, Resistor_SMD:R_0603_1608Metric_Pad1.05x0.95mm_HandSolder, F.Cu at (140.6, 49.1)
- added R23: 20k, Resistor_SMD:R_0603_1608Metric_Pad1.05x0.95mm_HandSolder, F.Cu at (137.7, 49.1)
- added R24: 2k9, Resistor_SMD:R_0603_1608Metric_Pad1.05x0.95mm_HandSolder, F.Cu at (135.0, 49.0)
- added R25: 100, Resistor_SMD:R_0603_1608Metric_Pad1.05x0.95mm_HandSolder, F.Cu at (132.3, 49.0)
- added R26: 100k, Resistor_SMD:R_0603_1608Metric_Pad1.05x0.95mm_HandSolder, F.Cu at (182.8, 26.9)
- added R27: 4k7, Resistor_SMD:R_0603_1608Metric_Pad1.05x0.95mm_HandSolder, F.Cu at (213.5, 35.6)
- added R3: 7k6, Resistor_SMD:R_0603_1608Metric_Pad1.05x0.95mm_HandSolder, F.Cu at (160.1, 42.1)
- added R4: 7k6, Resistor_SMD:R_0603_1608Metric_Pad1.05x0.95mm_HandSolder, F.Cu at (157.3, 42.2)
- added R5: 7k6, Resistor_SMD:R_0603_1608Metric_Pad1.05x0.95mm_HandSolder, F.Cu at (154.6, 42.2)
- added R6: 7k6, Resistor_SMD:R_0603_1608Metric_Pad1.05x0.95mm_HandSolder, F.Cu at (151.9, 42.2)
- added R7: 7k6, Resistor_SMD:R_0603_1608Metric_Pad1.05x0.95mm_HandSolder, F.Cu at (149.0, 42.1)
- added R8: 7k6, Resistor_SMD:R_0603_1608Metric_Pad1.05x0.95mm_HandSolder, F.Cu at (146.1, 42.2)
- added R9: 7k6, Resistor_SMD:R_0603_1608Metric_Pad1.05x0.95mm_HandSolder, F.Cu at (143.4, 42.2)
- added U2: L7805, Package_TO_SOT_THT:TO-220-3_Horizontal_TabDown, F.Cu at (165.7, 30.3)
- R1: footprint Resistor_SMD:R_0603_1608Metric -> Resistor_SMD:R_0603_1608Metric_Pad1.05x0.95mm_HandSolder
- moved J2 350.9 mm to (205.4, 52.3), turned to 270 degrees
- moved J3 306.5 mm to (167.3, 39.6)
- moved SW1 256.1 mm to (221.3, 49.4), turned to 90 degrees
- moved A1 253.4 mm to (191.4, 28.9), turned to 90 degrees
- moved J1 243.8 mm to (90.2, 52.3), turned to 90 degrees
- moved R1 234.6 mm to (90.2, 48.4), turned to 270 degrees
- moved U1 223.5 mm to (143.0, 31.4), turned to 180 degrees
- moved J5-~E1 45.6 mm to (134.5, 20.8)
- moved J15 33.4 mm to (90.2, 20.8)
- moved J4 32.8 mm to (144.2, 20.9)
Connections:
- A1 pad 21: (no net) -> /testpoints/TP5
- A1 pad 29: (no net) -> /RELAY/Relay_Driver
- A1 pad 30: (no net) -> /testpoints/TP4
- A1 pad 31: Net-(A1-Pad31) -> (no net)
- J15 pad 12: Net-(J15-Pad12) -> /testpoints/TP5
- J15 pad 15: Net-(J15-Pad15) -> GND
- J15 pad 4: Net-(J15-Pad4) -> /testpoints/TP4
- J17-TP3 pad 1: Net-(J15-Pad4) -> /testpoints/TP4
- J25-TP18 pad 1: Net-(J15-Pad12) -> /testpoints/TP5
- J4-TP16 pad 1: Net-(J4-TP16-Pad1) -> /4067/RELAY
- J7-TP27 pad 1: Net-(J7-TP27-Pad1) -> Net-(D1-Pad1)
- U1 pad 1: /4067/A0(Vref) -> Net-(R26-Pad1)
- U1 pad 2: Net-(J11-TP7-Pad1) -> Net-(R21-Pad2)
- U1 pad 20: Net-(J15-TP20-Pad1) -> Net-(R13-Pad1)
- U1 pad 21: Net-(J14-TP17-Pad1) -> Net-(R12-Pad1)
- U1 pad 22: Net-(J13-TP23-Pad1) -> Net-(R11-Pad1)
- U1 pad 23: Net-(J12-TP14-Pad1) -> Net-(R10-Pad1)
- U1 pad 3: Net-(J10-TP22-Pad1) -> Net-(R20-Pad2)
- U1 pad 4: Net-(J9-TP19-Pad1) -> Net-(R19-Pad2)
- U1 pad 5: Net-(J8-TP13-Pad1) -> Net-(R18-Pad2)
- U1 pad 6: Net-(J7-TP27-Pad1) -> Net-(R17-Pad2)
- U1 pad 7: Net-(J6-TP21-Pad1) -> Net-(R16-Pad2)
- U1 pad 8: Net-(J5-TP8-Pad1) -> Net-(R15-Pad2)
- U1 pad 9: Net-(J4-TP16-Pad1) -> Net-(R14-Pad2)
Routing:
- net /testpoints/TP4: track 0.00 -> 252.1 mm, vias 0 -> 6
- net +5V: track 0.00 -> 244.9 mm, vias 0 -> 10
- net /testpoints/TP5: track 0.00 -> 243.8 mm, vias 0 -> 2
- net Net-(J1-Pad3): track 0.00 -> 189.6 mm, vias 0 -> 1
- net Net-(J1-Pad4): track 0.00 -> 185.5 mm, vias 0 -> 1
- net Net-(J15-Pad13): track 0.00 -> 185.0 mm
- net Net-(J1-Pad5): track 0.00 -> 180.3 mm, vias 0 -> 1
- net Net-(J15-Pad8): track 0.00 -> 179.3 mm, vias 0 -> 5
- net Net-(J1-Pad6): track 0.00 -> 175.7 mm, vias 0 -> 1
- net Net-(J15-Pad2): track 0.00 -> 172.9 mm, vias 0 -> 4
- net Net-(J1-Pad7): track 0.00 -> 171.0 mm, vias 0 -> 1
- net Net-(J15-Pad3): track 0.00 -> 168.8 mm, vias 0 -> 6
- net Net-(J15-Pad5): track 0.00 -> 166.3 mm, vias 0 -> 4
- net Net-(J1-Pad8): track 0.00 -> 163.7 mm, vias 0 -> 1
- net Net-(J15-Pad14): track 0.00 -> 159.0 mm, vias 0 -> 2
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Other:
- board size 158.3 x 150.4 mm -> 158.3 x 160.4 mm
- copper layers 4 -> 2
- board text added: "DCTMM_CC-TESTER V0.1 20/02/2020"
