File: HW/carecasetester/display.sch (KiCad schematic (older format))
At the start: 4 parts, among them J1 Conn_01x16_Female, J2 Conn_01x16_Female, J3 Conn_01x04_Female

Commit message: cc-tester v0.1 gerber filser genereret og 1. print bestilles
Parts:
- R1: footprint Resistor_SMD:R_0603_1608Metric -> Resistor_SMD:R_0603_1608Metric_Pad1.05x0.95mm_HandSolder
Changed lines of the file:
@@
 $Descr A4 11693 8268
 encoding utf-8
-Sheet 2 5
+Sheet 2 6
 Title ""
 Date ""
@@
 F 0 "R1" H 8359 1771 50  0000 L CNN
 F 1 "180" H 8359 1680 50  0000 L CNN
-F 2 "Resistor_SMD:R_0603_1608Metric" H 8300 1725 50  0001 C CNN
+F 2 "Resistor_SMD:R_0603_1608Metric_Pad1.05x0.95mm_HandSolder" H 8300 1725 50  0001 C CNN
 F 3 "~" H 8300 1725 50  0001 C CNN
 	1    8300 1725
