File: HW/carecasetester/4067.sch (KiCad schematic (older format))
At the start: 40 parts, among them J10-TP22 Conn_01x01_Male, J11-TP7 Conn_01x01_Male, J12-TP14 Conn_01x01_Male, J13-TP23 Conn_01x01_Male, J14-TP17 Conn_01x01_Male, J15-TP20 Conn_01x01_Male, J16-TP24 Conn_01x01_Male, J4-TP16 Conn_01x01_Male, J5-TP8 Conn_01x01_Male, J5-~E1 Conn_01x02_Male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

Commit message: cc-tester v0.1 gerber filser genereret og 1. print bestilles
Parts:
- added R26: 100k, Resistor_SMD:R_0603_1608Metric_Pad1.05x0.95mm_HandSolder, symbol Device:R_Small
- D1: value 1N4001 -> 1N4001-B
- R10, R11, R12, R13, R14, R15, R16, R17, R18, R19, R2, R20, R21, R22, R23, R24, R25, R3, R4, R5, R6, R7, R8, R9: footprint (none) -> Resistor_SMD:R_0603_1608Metric_Pad1.05x0.95mm_HandSolder
Connections:
- net A0(Vref): now also R26.2; no longer U1.1 (COM)
- net +12V renamed RELAY
- new net: R26.1, U1.1 (COM)
Changed lines of the file:
@@
 $Descr A4 11693 8268
 encoding utf-8
-Sheet 3 5
+Sheet 3 6
 Title ""
 Date ""
@@
 A0(Vref)
 Wire Wire Line
-	5450 2650 4775 2650
+	5450 2650 5250 2650
 Text HLabel 4750 3050 0    50   Input ~ 0
 D2
@@
 F 0 "R2" H 6584 4696 50  0000 L CNN
 F 1 "7k6" H 6584 4605 50  0000 L CNN
-F 2 "" H 6525 4650 50  0001 C CNN
+F 2 "Resistor_SMD:R_0603_1608Metric_Pad1.05x0.95mm_HandSolder" H 6525 4650 50  0001 C CNN
 F 3 "~" H 6525 4650 50  0001 C CNN
 	1    6525 4650
@@
 F 0 "R3" H 6834 4696 50  0000 L CNN
 F 1 "7k6" H 6834 4605 50  0000 L CNN
-F 2 "" H 6775 4650 50  0001 C CNN
+F 2 "Resistor_SMD:R_0603_1608Metric_Pad1.05x0.95mm_HandSolder" H 6775 4650 50  0001 C CNN
 F 3 "~" H 6775 4650 50  0001 C CNN
 	1    6775 4650
@@
 F 0 "R4" H 7084 4696 50  0000 L CNN
 F 1 "7k6" H 7084 4605 50  0000 L CNN
-F 2 "" H 7025 4650 50  0001 C CNN
+F 2 "Resistor_SMD:R_0603_1608Metric_Pad1.05x0.95mm_HandSolder" H 7025 4650 50  0001 C CNN
 F 3 "~" H 7025 4650 50  0001 C CNN
 	1    7025 4650
@@
 F 0 "R5" H 7334 4696 50  0000 L CNN
 F 1 "7k6" H 7334 4605 50  0000 L CNN
-F 2 "" H 7275 4650 50  0001 C CNN
+F 2 "Resistor_SMD:R_0603_1608Metric_Pad1.05x0.95mm_HandSolder" H 7275 4650 50  0001 C CNN
 F 3 "~" H 7275 4650 50  0001 C CNN
 	1    7275 4650
@@
 F 0 "R6" H 7584 4696 50  0000 L CNN
 F 1 "7k6" H 7584 4605 50  0000 L CNN
-F 2 "" H 7525 4650 50  0001 C CNN
+F 2 "Resistor_SMD:R_0603_1608Metric_Pad1.05x0.95mm_HandSolder" H 7525 4650 50  0001 C CNN
 F 3 "~" H 7525 4650 50  0001 C CNN
 	1    7525 4650
@@
 F 0 "R7" H 7834 4696 50  0000 L CNN
 F 1 "7k6" H 7834 4605 50  0000 L CNN
-F 2 "" H 7775 4650 50  0001 C CNN
+F 2 "Resistor_SMD:R_0603_1608Metric_Pad1.05x0.95mm_HandSolder" H 7775 4650 50  0001 C CNN
 F 3 "~" H 7775 4650 50  0001 C CNN
 	1    7775 4650
@@
 F 0 "R8" H 8084 4696 50  0000 L CNN
 F 1 "7k6" H 8084 4605 50  0000 L CNN
-F 2 "" H 8025 4650 50  0001 C CNN
+F 2 "Resistor_SMD:R_0603_1608Metric_Pad1.05x0.95mm_HandSolder" H 8025 4650 50  0001 C CNN
 F 3 "~" H 8025 4650 50  0001 C CNN
 	1    8025 4650
@@
 F 0 "R9" H 8334 4696 50  0000 L CNN
 F 1 "7k6" H 8334 4605 50  0000 L CNN
-F 2 "" H 8275 4650 50  0001 C CNN
+F 2 "Resistor_SMD:R_0603_1608Metric_Pad1.05x0.95mm_HandSolder" H 8275 4650 50  0001 C CNN
 F 3 "~" H 8275 4650 50  0001 C CNN
 	1    8275 4650
@@
 F 0 "R10" H 8584 4696 50  0000 L CNN
 F 1 "7k6" H 8584 4605 50  0000 L CNN
-F 2 "" H 8525 4650 50  0001 C CNN
+F 2 "Resistor_SMD:R_0603_1608Metric_Pad1.05x0.95mm_HandSolder" H 8525 4650 50  0001 C CNN
 F 3 "~" H 8525 4650 50  0001 C CNN
 	1    8525 4650
@@
 F 0 "R11" H 8834 4696 50  0000 L CNN
 F 1 "7k6" H 8834 4605 50  0000 L CNN
-F 2 "" H 8775 4650 50  0001 C CNN
+F 2 "Resistor_SMD:R_0603_1608Metric_Pad1.05x0.95mm_HandSolder" H 8775 4650 50  0001 C CNN
 F 3 "~" H 8775 4650 50  0001 C CNN
 	1    8775 4650
@@
 F 0 "R12" H 9084 4696 50  0000 L CNN
 F 1 "7k6" H 9084 4605 50  0000 L CNN
-F 2 "" H 9025 4650 50  0001 C CNN
+F 2 "Resistor_SMD:R_0603_1608Metric_Pad1.05x0.95mm_HandSolder" H 9025 4650 50  0001 C CNN
 F 3 "~" H 9025 4650 50  0001 C CNN
 	1    9025 4650
@@
 F 0 "R13" H 9334 4696 50  0000 L CNN
 F 1 "7k6" H 9334 4605 50  0000 L CNN
-F 2 "" H 9275 4650 50  0001 C CNN
+F 2 "Resistor_SMD:R_0603_1608Metric_Pad1.05x0.95mm_HandSolder" H 9275 4650 50  0001 C CNN
 F 3 "~" H 9275 4650 50  0001 C CNN
 	1    9275 4650
@@
 Wire Wire Line
 	9025 4025 9275 4025
-Wire Wire Line
-	9275 4550 9275 4225
 $Comp
 L Device:R_Small R14
@@
 F 0 "R14" V 9375 1925 50  0000 C CNN
 F 1 "20k" V 9270 1925 50  0000 C CNN
-F 2 "" H 9375 1925 50  0001 C CNN
+F 2 "Resistor_SMD:R_0603_1608Metric_Pad1.05x0.95mm_HandSolder" H 9375 1925 50  0001 C CNN
 F 3 "~" H 9375 1925 50  0001 C CNN
 	1    9375 1925
@@
 F 0 "R15" V 9375 2125 50  0000 C CNN
 F 1 "20k" V 9270 2125 50  0000 C CNN
-F 2 "" H 9375 2125 50  0001 C CNN
+F 2 "Resistor_SMD:R_0603_1608Metric_Pad1.05x0.95mm_HandSolder" H 9375 2125 50  0001 C CNN
 F 3 "~" H 9375 2125 50  0001 C CNN
 	1    9375 2125
@@
 F 0 "R21" V 9375 3375 50  0000 C CNN
 F 1 "20k" V 9270 3375 50  0000 C CNN
-F 2 "" H 9375 3375 50  0001 C CNN
+F 2 "Resistor_SMD:R_0603_1608Metric_Pad1.05x0.95mm_HandSolder" H 9375 3375 50  0001 C CNN
 F 3 "~" H 9375 3375 50  0001 C CNN
 	1    9375 3375
@@
 F 0 "R22" V 9375 3575 50  0000 C CNN
 F 1 "20k" V 9270 3575 50  0000 C CNN
-F 2 "" H 9375 3575 50  0001 C CNN
+F 2 "Resistor_SMD:R_0603_1608Metric_Pad1.05x0.95mm_HandSolder" H 9375 3575 50  0001 C CNN
 F 3 "~" H 9375 3575 50  0001 C CNN
 	1    9375 3575
@@
 F 0 "R23" V 9375 3825 50  0000 C CNN
 F 1 "20k" V 9270 3825 50  0000 C CNN
-F 2 "" H 9375 3825 50  0001 C CNN
+F 2 "Resistor_SMD:R_0603_1608Metric_Pad1.05x0.95mm_HandSolder" H 9375 3825 50  0001 C CNN
 F 3 "~" H 9375 3825 50  0001 C CNN
 	1    9375 3825
@@
 F 0 "R16" V 9375 2325 50  0000 C CNN
 F 1 "3k9" V 9270 2325 50  0000 C CNN
-F 2 "" H 9375 2325 50  0001 C CNN
+F 2 "Resistor_SMD:R_0603_1608Metric_Pad1.05x0.95mm_HandSolder" H 9375 2325 50  0001 C CNN
 F 3 "~" H 9375 2325 50  0001 C CNN
 	1    9375 2325
@@
 F 0 "R19" V 9375 2950 50  0000 C CNN
 F 1 "3k9" V 9270 2950 50  0000 C CNN
-F 2 "" H 9375 2950 50  0001 C CNN
+F 2 "Resistor_SMD:R_0603_1608Metric_Pad1.05x0.95mm_HandSolder" H 9375 2950 50  0001 C CNN
 F 3 "~" H 9375 2950 50  0001 C CNN
 	1    9375 2950
@@
 F 0 "R20" V 9375 3175 50  0000 C CNN
 F 1 "3k9" V 9270 3175 50  0000 C CNN
-F 2 "" H 9375 3175 50  0001 C CNN
+F 2 "Resistor_SMD:R_0603_1608Metric_Pad1.05x0.95mm_HandSolder" H 9375 3175 50  0001 C CNN
 F 3 "~" H 9375 3175 50  0001 C CNN
 	1    9375 3175
@@
 F 0 "R17" V 9375 2550 50  0000 C CNN
 F 1 "2k9" V 9270 2550 50  0000 C CNN
-F 2 "" H 9375 2550 50  0001 C CNN
+F 2 "Resistor_SMD:R_0603_1608Metric_Pad1.05x0.95mm_HandSolder" H 9375 2550 50  0001 C CNN
 F 3 "~" H 9375 2550 50  0001 C CNN
 	1    9375 2550
@@
 F 0 "R18" V 9375 2750 50  0000 C CNN
 F 1 "2k9" V 9270 2750 50  0000 C CNN
-F 2 "" H 9375 2750 50  0001 C CNN
+F 2 "Resistor_SMD:R_0603_1608Metric_Pad1.05x0.95mm_HandSolder" H 9375 2750 50  0001 C CNN
 F 3 "~" H 9375 2750 50  0001 C CNN
 	1    9375 2750
@@
 F 0 "R24" V 9375 4025 50  0000 C CNN
 F 1 "2k9" V 9270 4025 50  0000 C CNN
-F 2 "" H 9375 4025 50  0001 C CNN
+F 2 "Resistor_SMD:R_0603_1608Metric_Pad1.05x0.95mm_HandSolder" H 9375 4025 50  0001 C CNN
 F 3 "~" H 9375 4025 50  0001 C CNN
 	1    9375 4025
@@
 F 0 "R25" V 9375 4225 50  0000 C CNN
 F 1 "100" V 9270 4225 50  0000 C CNN
-F 2 "" H 9375 4225 50  0001 C CNN
+F 2 "Resistor_SMD:R_0603_1608Metric_Pad1.05x0.95mm_HandSolder" H 9375 4225 50  0001 C CNN
 F 3 "~" H 9375 4225 50  0001 C CNN
 	1    9375 4225
@@
 Wire Wire Line
 	9775 2125 9475 2125
-Wire Wire Line
-	9475 1925 9600 1925
-$Comp
-L power:+12V #PWR01
-U 1 1 5E453E7D
-P 9600 1925
-F 0 "#PWR01" H 9600 1775 50  0001 C CNN
-F 1 "+12V" H 9615 2098 50  0000 C CNN
-F 2 "" H 9600 1925 50  0001 C CNN
-F 3 "" H 9600 1925 50  0001 C CNN
-	1    9600 1925
-	1    0    0    -1
-$EndComp
-Connection ~ 9600 1925
-Wire Wire Line
-	9600 1925 9775 1925
 Wire Wire Line
 	9475 2550 9675 2550
@@
 P 10775 2650
 F 0 "D1" H 10925 2700 50  0000 C CNN
-F 1 "1N4001" H 11000 2600 50  0000 C CNN
+F 1 "1N4001-B" H 11000 2600 50  0000 C CNN
 F 2 "Diode_THT:D_DO-41_SOD81_P10.16mm_Horizontal" H 10775 2475 50  0001 C CNN
 F 3 "http://www.vishay.com/docs/88503/1n4001.pdf" H 10775 2650 50  0001 C CNN
@@
 Wire Wire Line
 	11025 2650 11025 2625
+Connection ~ 9275 4225
+Wire Wire Line
+	9275 4225 9275 4550
+$Comp
+L Device:R_Small R26
+U 1 1 5E3CC792
+P 5150 2650
+F 0 "R26" V 4954 2650 50  0000 C CNN
+F 1 "100k" V 5045 2650 50  0000 C CNN
+F 2 "Resistor_SMD:R_0603_1608Metric_Pad1.05x0.95mm_HandSolder" H 5150 2650 50  0001 C CNN
+F 3 "~" H 5150 2650 50  0001 C CNN
+	1    5150 2650
+	0    1    1    0
+$EndComp
+Wire Wire Line
+	5050 2650 4775 2650
+Wire Wire Line
+	9475 1925 9600 1925
+Text HLabel 9600 1600 1    50   Input ~ 0
+RELAY
+Wire Wire Line
+	9600 1600 9600 1925
+Connection ~ 9600 1925
+Wire Wire Line
+	9600 1925 9775 1925
 $EndSCHEMATC

Commit message: V0.22 gerbers
2nd relay added and all should now be ready to order
Connections:
- net +5V: no longer D1.2 (A)
- net RELAY renamed RELAY12V
- new net RELAYBAT: D1.2 (A)
Changed lines of the file:
@@
 Wire Wire Line
 	9675 2550 9775 2550
-$Comp
-L power:+5V #PWR02
-U 1 1 5E464082
-P 11025 2625
-F 0 "#PWR02" H 11025 2475 50  0001 C CNN
-F 1 "+5V" H 11040 2798 50  0000 C CNN
-F 2 "" H 11025 2625 50  0001 C CNN
-F 3 "" H 11025 2625 50  0001 C CNN
-	1    11025 2625
-	1    0    0    -1
-$EndComp
 Wire Wire Line
 	10925 2650 11025 2650
@@
 	9475 1925 9600 1925
 Text HLabel 9600 1600 1    50   Input ~ 0
-RELAY
+RELAY12V
 Wire Wire Line
 	9600 1600 9600 1925
@@
 Wire Wire Line
 	9600 1925 9775 1925
+Text HLabel 11025 2625 1    50   Input ~ 0
+RELAYBAT
 $EndSCHEMATC
